File: nrf24l01_door_alarm.sch (KiCad schematic (older format))
At the start: 15 parts, among them J1 Conn_01x02_Male, J2 Conn_02x03_Odd_Even, Q1 2N7002, SW1 SW_Reed, U1 ATmega328P-AU, U2 NRF24L01_Breakout

Commit message: initial pcb layout
Parts:
- C1: footprint (none) -> Capacitor_THT:CP_Radial_D5.0mm_P2.50mm
- C2, C3, C4: footprint (none) -> Capacitor_SMD:C_0805_2012Metric_Pad1.15x1.40mm_HandSolder
- D1: footprint (none) -> LED_SMD:LED_0805_2012Metric_Pad1.15x1.40mm_HandSolder
- J1: footprint (none) -> Connector_PinHeader_2.54mm:PinHeader_1x02_P2.54mm_Vertical
- J2: footprint (none) -> Connector_PinHeader_2.54mm:PinHeader_2x03_P2.54mm_Vertical
- R1, R2, R3, R4: footprint (none) -> Resistor_SMD:R_0805_2012Metric_Pad1.15x1.40mm_HandSolder
- SW1: footprint (none) -> Connector_PinHeader_2.54mm:PinHeader_2x01_P2.54mm_Vertical
- U2: footprint RF_Module:nRF24L01_Breakout -> mysensor_radios:NRF24L01-SMD
Changed lines of the file:
@@
 F 0 "J1" H 1208 1831 50  0000 C CNN
 F 1 "Conn_01x02_Male" H 1208 1740 50  0000 C CNN
-F 2 "" H 1100 1650 50  0001 C CNN
+F 2 "Connector_PinHeader_2.54mm:PinHeader_1x02_P2.54mm_Vertical" H 1100 1650 50  0001 C CNN
 F 3 "~" H 1100 1650 50  0001 C CNN
 	1    1100 1650
@@
 F 0 "C1" H 1941 1796 50  0000 L CNN
 F 1 "100uF" H 1941 1705 50  0000 L CNN
-F 2 "" H 1850 1750 50  0001 C CNN
+F 2 "Capacitor_THT:CP_Radial_D5.0mm_P2.50mm" H 1850 1750 50  0001 C CNN
 F 3 "~" H 1850 1750 50  0001 C CNN
 	1    1850 1750
@@
 F 0 "C2" H 2292 1796 50  0000 L CNN
 F 1 "100nF" H 2292 1705 50  0000 L CNN
-F 2 "" H 2200 1750 50  0001 C CNN
+F 2 "Capacitor_SMD:C_0805_2012Metric_Pad1.15x1.40mm_HandSolder" H 2200 1750 50  0001 C CNN
 F 3 "~" H 2200 1750 50  0001 C CNN
 	1    2200 1750
@@
 F 0 "C3" H 2592 1796 50  0000 L CNN
 F 1 "100nF" H 2592 1705 50  0000 L CNN
-F 2 "" H 2500 1750 50  0001 C CNN
+F 2 "Capacitor_SMD:C_0805_2012Metric_Pad1.15x1.40mm_HandSolder" H 2500 1750 50  0001 C CNN
 F 3 "~" H 2500 1750 50  0001 C CNN
 	1    2500 1750
@@
 F 0 "C4" H 2842 1796 50  0000 L CNN
 F 1 "100nF" H 2842 1705 50  0000 L CNN
-F 2 "" H 2750 1750 50  0001 C CNN
+F 2 "Capacitor_SMD:C_0805_2012Metric_Pad1.15x1.40mm_HandSolder" H 2750 1750 50  0001 C CNN
 F 3 "~" H 2750 1750 50  0001 C CNN
 	1    2750 1750
@@
 F 0 "R3" H 8720 4546 50  0000 L CNN
 F 1 "47K" H 8720 4455 50  0000 L CNN
-F 2 "" V 8580 4500 50  0001 C CNN
+F 2 "Resistor_SMD:R_0805_2012Metric_Pad1.15x1.40mm_HandSolder" V 8580 4500 50  0001 C CNN
 F 3 "~" H 8650 4500 50  0001 C CNN
 	1    8650 4500
@@
 F 0 "R4" H 8270 4546 50  0000 L CNN
 F 1 "1M" H 8270 4455 50  0000 L CNN
-F 2 "" V 8130 4500 50  0001 C CNN
+F 2 "Resistor_SMD:R_0805_2012Metric_Pad1.15x1.40mm_HandSolder" V 8130 4500 50  0001 C CNN
 F 3 "~" H 8200 4500 50  0001 C CNN
 	1    8200 4500
@@
 F 0 "R2" V 5250 5700 50  0000 L CNN
 F 1 "1K" V 5450 5700 50  0000 L CNN
-F 2 "" V 5280 5750 50  0001 C CNN
+F 2 "Resistor_SMD:R_0805_2012Metric_Pad1.15x1.40mm_HandSolder" V 5280 5750 50  0001 C CNN
 F 3 "~" H 5350 5750 50  0001 C CNN
 	1    5350 5750
@@
 F 0 "D1" H 5843 5967 50  0000 C CNN
 F 1 "LED" H 5843 5876 50  0000 C CNN
-F 2 "" H 5850 5750 50  0001 C CNN
+F 2 "LED_SMD:LED_0805_2012Metric_Pad1.15x1.40mm_HandSolder" H 5850 5750 50  0001 C CNN
 F 3 "~" H 5850 5750 50  0001 C CNN
 	1    5850 5750
@@
 F 0 "J2" H 9750 1317 50  0000 C CNN
 F 1 "Conn_02x03_Odd_Even" H 9750 1226 50  0000 C CNN
-F 2 "" H 9700 1000 50  0001 C CNN
+F 2 "Connector_PinHeader_2.54mm:PinHeader_2x03_P2.54mm_Vertical" H 9700 1000 50  0001 C CNN
 F 3 "~" H 9700 1000 50  0001 C CNN
 	1    9700 1000
@@
 F 0 "SW1" H 8200 5472 50  0000 C CNN
 F 1 "SW_Reed" H 8200 5381 50  0000 C CNN
-F 2 "" H 8200 5250 50  0001 C CNN
+F 2 "Connector_PinHeader_2.54mm:PinHeader_2x01_P2.54mm_Vertical" H 8200 5250 50  0001 C CNN
 F 3 "~" H 8200 5250 50  0001 C CNN
 	1    8200 5250
@@
 F 0 "R1" V 5693 3350 50  0000 C CNN
 F 1 "10K" V 5784 3350 50  0000 C CNN
-F 2 "" V 5830 3350 50  0001 C CNN
+F 2 "Resistor_SMD:R_0805_2012Metric_Pad1.15x1.40mm_HandSolder" V 5830 3350 50  0001 C CNN
 F 3 "~" H 5900 3350 50  0001 C CNN
 	1    5900 3350
@@
 F 0 "U2" H 9030 2596 50  0000 L CNN
 F 1 "NRF24L01_Breakout" H 9030 2505 50  0000 L CNN
-F 2 "RF_Module:nRF24L01_Breakout" H 8800 3150 50  0001 L CIN
+F 2 "mysensor_radios:NRF24L01-SMD" H 8800 3150 50  0001 L CIN
 F 3 "http://www.nordicsemi.com/eng/content/download/2730/34105/file/nRF24L01_Product_Specification_v2_0.pdf" H 8650 2450 50  0001 C CNN
 	1    8650 2550
